File: kicad/ch32v004jm6-ds1302.kicad_pcb (KiCad board)
At the start: 2 copper layers, 24.1 x 38.1 mm, 10 parts, among them J2 Conn_01x03_Pin, SW1 SW_Push, U2 DS1302+, Y1 Crystal

Commit message: Update CAD data
Parts:
- removed J2: Conn_01x03_Pin, Connector_PinSocket_2.54mm:PinSocket_2x02_P2.54mm_Vertical
- added J1: Conn_01x04_Pin, Connector_PinSocket_2.54mm:PinSocket_2x02_P2.54mm_Vertical, F.Cu at (150.5, 66.0)
- added R1: R, Resistor_SMD:R_0603_1608Metric, F.Cu at (142.2, 66.7)
- added REF**: MountingHole_3.2mm_M3, MountingHole:MountingHole_3.2mm_M3, F.Cu at (151.1, 97.2)
- added REF**: MountingHole_3.2mm_M3, MountingHole:MountingHole_3.2mm_M3, F.Cu at (133.3, 65.4)
- added REF**: MountingHole_3.2mm_M3, MountingHole:MountingHole_3.2mm_M3, F.Cu at (133.3, 97.2)
- moved D1 1.56 mm to (139.7, 67.3)
- moved D2 1.27 mm to (144.8, 67.3)
- moved C1 1.27 mm to (137.2, 72.4)
- moved BT1 0.72 mm to (142.2, 81.2)
- moved C2 0.51 mm to (138.4, 87.5), turned to -90 degrees
Connections:
- BT1 pad 1: +3.3V -> +BATT
- SW1 pad 2: +3.3V -> +BATT
- U1 pad 3: Net-(D2-A) -> Net-(U1-PA2)
- U2 pad 8: +3.3V -> +BATT
Routing:
- net +BATT: track 0.00 -> 38.4 mm, vias 0 -> 1
- net +3.3V: track 86.0 -> 59.5 mm, vias 1 -> 0
- net Net-(D2-A): track 13.5 -> 2.30 mm
- net Net-(U1-PA2): track 0.00 -> 7.58 mm
- net Net-(J1-Pin_1): track 8.44 -> 7.47 mm
- net Net-(D1-A): track 3.03 -> 2.39 mm
- added copper zone on F.Cu, net +3.3V
Other:
- board text added: "+3.3V"
- board text added: "."
- board text added: "GND"
- board text added: "SWIO"
- board text added: "ver 0.1 @task_jp"
